Commit message: drop the project (hard 2 gen normal gait)

File: legged_gym/resources/robots/go1/urdf/go1.urdf (robot description, URDF)
Before this commit: robot go1, 46 links, 45 joints
Links:
- removed link FL_calf_rotor
- removed link FL_hip_rotor
- removed link FL_thigh_rotor
- removed link FR_calf_rotor
- removed link FR_hip_rotor
- removed link FR_thigh_rotor
- removed link RL_calf_rotor
- removed link RL_hip_rotor
- removed link RL_thigh_rotor
- removed link RR_calf_rotor
- removed link RR_hip_rotor
- removed link RR_thigh_rotor
- added link FL_thigh_shoulder
- added link FR_thigh_shoulder
- added link RL_thigh_shoulder
- added link RR_thigh_shoulder
- link FL_calf: mass 0.135862 -> 0.131
- link FL_hip: geometry visual mesh filename=../meshes/hip.dae scale=1 1 1
- link FR_calf: mass 0.135862 -> 0.131
- link FR_hip: geometry visual mesh filename=../meshes/hip.dae scale=1 1 1
- link RL_calf: mass 0.135862 -> 0.131
- link RL_hip: geometry visual mesh filename=../meshes/hip.dae scale=1 1 1
- link RR_calf: mass 0.135862 -> 0.131
- link RR_hip: geometry visual mesh filename=../meshes/hip.dae scale=1 1 1
- link imu_link: geometry visual box size=0.001 0.001 0.001
- link trunk: geometry collision box size=0.45 0.1935 0.05; visual mesh filename=../meshes/trunk.dae scale=1 1 1
Joints:
- removed joint FL_calf_rotor_joint
- removed joint FL_hip_rotor_joint
- removed joint FL_thigh_rotor_joint
- removed joint FR_calf_rotor_joint
- removed joint FR_hip_rotor_joint
- removed joint FR_thigh_rotor_joint
- removed joint RL_calf_rotor_joint
- removed joint RL_hip_rotor_joint
- removed joint RL_thigh_rotor_joint
- removed joint RR_calf_rotor_joint
- removed joint RR_hip_rotor_joint
- removed joint RR_thigh_rotor_joint
- added joint FL_hip_fixed: type fixed, parent FL_hip, child FL_thigh_shoulder, origin xyz=0 0.08 0 rpy=0 0 0
- added joint FR_hip_fixed: type fixed, parent FR_hip, child FR_thigh_shoulder, origin xyz=0 -0.08 0 rpy=0 0 0
- added joint RL_hip_fixed: type fixed, parent RL_hip, child RL_thigh_shoulder, origin xyz=0 0.08 0 rpy=0 0 0
- added joint RR_hip_fixed: type fixed, parent RR_hip, child RR_thigh_shoulder, origin xyz=0 -0.08 0 rpy=0 0 0
- joint FL_calf_joint: limit lower=-2.818 upper=-0.888 effort=35.55 velocity=20.06 -> lower=-2.72271363311 upper=-0.837758040957 effort=23.7 velocity=30.1
- joint FL_hip_joint: limit lower=-0.863 upper=0.863 effort=23.7 velocity=30.1 -> lower=-1.0471975512 upper=1.0471975512 effort=23.7 velocity=30.1
- joint FL_thigh_joint: limit lower=-0.686 upper=4.501 effort=23.7 velocity=30.1 -> lower=-0.663225115758 upper=2.96705972839 effort=23.7 velocity=30.1
- joint FR_calf_joint: limit lower=-2.818 upper=-0.888 effort=35.55 velocity=20.06 -> lower=-2.72271363311 upper=-0.837758040957 effort=23.7 velocity=30.1
- joint FR_hip_joint: limit lower=-0.863 upper=0.863 effort=23.7 velocity=30.1 -> lower=-1.0471975512 upper=1.0471975512 effort=23.7 velocity=30.1
- joint FR_thigh_joint: limit lower=-0.686 upper=4.501 effort=23.7 velocity=30.1 -> lower=-0.663225115758 upper=2.96705972839 effort=23.7 velocity=30.1
- joint RL_calf_joint: limit lower=-2.818 upper=-0.888 effort=35.55 velocity=20.06 -> lower=-2.72271363311 upper=-0.837758040957 effort=23.7 velocity=30.1
- joint RL_hip_joint: limit lower=-0.863 upper=0.863 effort=23.7 velocity=30.1 -> lower=-1.0471975512 upper=1.0471975512 effort=23.7 velocity=30.1
- joint RL_thigh_joint: limit lower=-0.686 upper=4.501 effort=23.7 velocity=30.1 -> lower=-0.663225115758 upper=2.96705972839 effort=23.7 velocity=30.1
- joint RR_calf_joint: limit lower=-2.818 upper=-0.888 effort=35.55 velocity=20.06 -> lower=-2.72271363311 upper=-0.837758040957 effort=23.7 velocity=30.1
- joint RR_hip_joint: limit lower=-0.863 upper=0.863 effort=23.7 velocity=30.1 -> lower=-1.0471975512 upper=1.0471975512 effort=23.7 velocity=30.1
- joint RR_thigh_joint: limit lower=-0.686 upper=4.501 effort=23.7 velocity=30.1 -> lower=-0.663225115758 upper=2.96705972839 effort=23.7 velocity=30.1
- joint camera_joint_chin: origin xyz=0.2522 0.0125 -0.0436 rpy=3.141592653589793 1.5707963267948966 0 -> xyz=0.2522 0.0125 -0.0436 rpy=3.14159265359 1.57079632679 0
- joint camera_joint_face: origin xyz=0.2785 0.0125 0.0167 rpy=3.141592653589793 0 0 -> xyz=0.2785 0.0125 0.0167 rpy=3.14159265359 0 0
- joint camera_joint_left: origin xyz=-0.066 0.082 -0.0176 rpy=3.141592653589793 0.2618 1.5707963267948966 -> xyz=-0.066 0.082 -0.0176 rpy=3.14159265359 0.2618 1.57079632679
- joint camera_joint_rearDown: origin xyz=-0.0825 0.0125 -0.04365 rpy=3.141592653589793 1.5707963267948966 0 -> xyz=-0.0825 0.0125 -0.04365 rpy=3.14159265359 1.57079632679 0
- joint camera_joint_right: origin xyz=-0.041 -0.082 -0.0176 rpy=3.141592653589793 0.2618 -1.5707963267948966 -> xyz=-0.041 -0.082 -0.0176 rpy=3.14159265359 0.2618 -1.57079632679
- joint camera_optical_joint_chin: origin xyz=0 0 0 rpy=-1.5707963267948966 0 -1.5707963267948966 -> xyz=0 0 0 rpy=-1.57079632679 0 -1.57079632679
- joint camera_optical_joint_face: origin xyz=0 0 0 rpy=-1.5707963267948966 0 -1.5707963267948966 -> xyz=0 0 0 rpy=-1.57079632679 0 -1.57079632679
- joint camera_optical_joint_left: origin xyz=0 0 0 rpy=-1.5707963267948966 0 -1.5707963267948966 -> xyz=0 0 0 rpy=-1.57079632679 0 -1.57079632679
- joint camera_optical_joint_rearDown: origin xyz=0 0 0 rpy=-1.5707963267948966 0 -1.5707963267948966 -> xyz=0 0 0 rpy=-1.57079632679 0 -1.57079632679
- joint camera_optical_joint_right: origin xyz=0 0 0 rpy=-1.5707963267948966 0 -1.5707963267948966 -> xyz=0 0 0 rpy=-1.57079632679 0 -1.57079632679
- joint ultraSound_joint_left: origin xyz=-0.0535  0.0826 0.00868 rpy=0 0.2618 1.5707963267948966 -> xyz=-0.0535  0.0826 0.00868 rpy=0 0.2618 1.57079632679
- joint ultraSound_joint_right: origin xyz=-0.0535 -0.0826 0.00868 rpy=0 0.2618 -1.5707963267948966 -> xyz=-0.0535 -0.0826 0.00868 rpy=0 0.2618 -1.57079632679
